File: cooker-swarm-node-hardware-components.sch (KiCad schematic (older format))
At the start: 36 parts, among them J1 Conn_ARM_JTAG_SWD_10, J4 USB_B_Micro, X1 32MHz, 8pF, X2 32,768kHz, 9pF

Commit message: use MCP6002 opamp
Parts:
- added AE2: Antenna_Shield, Connector_Coaxial:U.FL_Molex_MCRF_73412-0110_Vertical, symbol Device:Antenna_Shield
- added C27: N.C., Capacitor_SMD:C_0402_1005Metric, symbol Device:C
- added C28: 100n, Capacitor_SMD:C_0402_1005Metric, symbol Device:C
- added R13, R14: 0, Resistor_SMD:R_0402_1005Metric, symbol Device:R
- added R15: 10k, Resistor_SMD:R_0402_1005Metric, symbol Device:R
Connections:
- net GND: now also AE2.2 (Shield), C27.1, C28.2, R15.1
- net at C7.1, L3.1: now also R13.1, R14.2; no longer AE1.1 (A), C4.1
- net at J4.6 (Shield): now also C28.1, R15.2
- new net: AE1.1 (A), C4.1, R14.1
- new net: AE2.1 (A), C27.2, R13.2
- no-connect marks 4 -> 3
Other:
- moved on the sheet: AE1, C11, C4, C7, L3
